Commit message: fix: update URDF joint limits for joint2, joint3, and joint5 to standard industrial limits of ±180 degrees (Math.PI) to allow convergence to target panel coordinates

File: vantage-sim/public/robot/arm.urdf (robot description, URDF)
Before this commit: robot vantage_arm, 8 links, 7 joints
Joints:
- joint joint2: limit lower=-1.5708 upper=1.5708 effort=100 velocity=1.0 -> lower=-3.14159 upper=3.14159 effort=100 velocity=1.0
- joint joint3: limit lower=-1.5708 upper=1.5708 effort=100 velocity=1.0 -> lower=-3.14159 upper=3.14159 effort=100 velocity=1.0
- joint joint5: limit lower=-1.5708 upper=1.5708 effort=50 velocity=1.5 -> lower=-3.14159 upper=3.14159 effort=50 velocity=1.5
